File: Hardware/key_matrix.kicad_sch (KiCad schematic)
At the start: 84 parts, among them SW1 ESC, SW10 TAB, SW11 Q, SW12 W, SW13 E, SW14 R, SW15 T, SW16 NA, SW17 M1, SW18 CAPS, SW19 A, SW2 `, SW20 S, SW21 D, SW22 F, SW23 G, SW24 NA, SW25 M2, SW26 M3, SW28 SHIFT, SW29 CTRL, SW3 1, SW30 Rot_Enc, SW31 Z, SW32 WIN, SW34 X, SW35 FN, SW37 C, SW38 ALT, SW4 2, SW40 V, SW41 SPACE, SW43 B, SW44 DEL, SW46 NA, SW47 NA, SW5 3, SW6 4, SW7 5, SW8 6, SW9 M0

Commit message: added mounting holes
Parts:
- SW1, SW2: LCSC (none) -> C41430893
Changed lines of the file:
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@@
 			)
 		)
+		(property "LCSC" "C41430893"
+			(at 218.44 86.36 0)
+			(effects
+				(font
+					(size 1.27 1.27)
+				)
+				(hide yes)
+			)
+		)
 		(pin "2"
 		)
@@
 			(at 203.2 86.36 0)
 			(effects
+				(font
+					(size 1.27 1.27)
+				)
+				(hide yes)
+			)
+		)
+		(property "LCSC" "C41430893"
+			(at 203.2 86.36 0)
+			(effects

Commit message: Add LCSC part numbers and new resistor to PCB
Added LCSC part numbers to multiple components in hornet_kb.kicad_pcb for improved BOM generation. Introduced a new 500Ω resistor (R11) and updated net assignments for Q1 and D27. Modified .gitignore to exclude backup and auto-save files, and removed obsolete backup files from Hardware/hornet_kb-backups. Made symbol and footprint tweaks in Custom_sym.kicad_sym.
Parts:
- D1, D10, D11, D12, D13, D14, D15, D17, D18, D19, D2, D20, D21, D22, D23, D25, D26, D28, D29, D3, D31, D32, D34, D35, D37, D38, D4, D40, D41, D43, D44, D5, D6, D7, D8, D9: LCSC (none) -> C917030
- SW10, SW11, SW12, SW13, SW14, SW15, SW17, SW18, SW19, SW20, SW21, SW22, SW23, SW25, SW26, SW28, SW29, SW3, SW30, SW31, SW32, SW34, SW35, SW37, SW38, SW4, SW40, SW41, SW43, SW44, SW5, SW6, SW7, SW8, SW9: LCSC (none) -> C41430893
Other:
- moved on the sheet: D1, D10, D11, D12, D13, D14, D15, D16, D17, D18, D19, D2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

Commit message: Added LCSC part defs
Parts:
- R14, R15, R3: LCSC (none) -> C25804
