File: Hardware/hornet_kb.kicad_pcb (KiCad board)
At the start: 4 copper layers, 199.5 x 120.1 mm, 157 parts, among them J1 Conn_ST_STDC14, J10 USB_C_Receptacle_USB2.0, J2 Conn_01x03, Q1 BTS4140N, SW1 ESC, SW10 TAB, SW11 Q, SW12 W, SW13 E, SW14 R, SW15 T, SW17 M1, SW18 CAPS, SW19 A, SW2 `, SW20 S, SW21 D, SW22 F, SW23 G, SW25 M2, SW26 M3, SW27 SW_DPDT_x2, SW28 SHIFT, SW29 CTRL, SW3 1, SW30 Rot_Enc, SW31 Z, SW32 WIN, SW34 X, SW35 FN, SW37 C, SW38 ALT, SW4 2, SW40 V, SW41 SPACE, SW43 B, SW44 DEL, SW5 3, SW6 4, SW7 5, SW8 6, SW9 M0, SW98 SW_Push, U1 nRF52840, U2 BQ24040, U3 BQ51050BRHL, U5 TPS2116DRL, Y1 32.768kHz, Y3 32Mhz

Commit message: Final Commits before production
Parts:
- moved L1 5.03 mm to (154.0, 39.2), turned to 0 degrees
- moved J2 2.57 mm to (261.2, 61.0), turned to 90 degrees
Routing:
- net +BATT: track 119.2 -> 130.9 mm
- net Net-(U3-AC2): track 139.2 -> 146.2 mm
- net /Power Management/BATT_NTC: track 12.5 -> 15.3 mm
- net GND: track 223.3 -> 221.3 mm
- net Net-(C13-Pad1): track 132.8 -> 131.5 mm

Commit message: Small adjustments
Routing:
- net +BATT: track 130.9 -> 129.0 mm
